File: hardware/mono_panel_32x32_v2/mono_panel_32x32_v2.kicad_pcb (KiCad board)
At the start: 4 copper layers, 256 x 256 mm, 1040 parts

Commit message: mono_panel_32x32_v2: replace 0.125 mm staircase routes with any-angle straight runs + tangent arcs; thermal fix; gates 0; fab + renders regenerated
Routing:
- net COL_26: track 340.0 -> 333.7 mm
- net COL_06: track 444.9 -> 439.9 mm
- net COL_30: track 369.4 -> 365.7 mm
- net COL_28: track 352.8 -> 349.7 mm
- net ROW_21: track 367.6 -> 364.6 mm
- net ROW_23: track 382.5 -> 379.5 mm
- net COL_07: track 433.5 -> 436.4 mm, vias 33 -> 34
- net ROW_25: track 397.3 -> 394.4 mm
- net COL_31: track 376.0 -> 378.7 mm, vias 33 -> 34
- net COL_09: track 421.0 -> 423.6 mm
- net ROW_19: track 352.2 -> 349.7 mm
- net ID_3V3: track 16.3 -> 14.0 mm
- net COL_02: track 473.9 -> 471.7 mm
- net ROW_24: track 387.2 -> 389.2 mm
- net ROW_22: track 372.3 -> 374.3 mm
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